Commit message: change model and nao parameters to match 3DSim

File: resources/robots/nao/urdf/nao_no_fingers.urdf (robot description, URDF)
Before this commit: robot NaoH25V50, 79 links, 78 joints
Joints:
- joint LHand: type fixed -> revolute
- joint LWristYaw: type fixed -> revolute
- joint RHand: type fixed -> revolute
- joint RWristYaw: type fixed -> revolute
